Commit message: made the test stand a slider and separated sim and hardware xacros

File: src/rl12dof_urdf_description/urdf/materials.xacro (robot description, xacro)
@@ -4,3 +4,9 @@
   <color rgba="0.700 0.700 0.700 1.000"/>
 </material>
+<material name="blue">
+  <color rgba="0 0 1 1"/>
+</material>
+<material name="red">
+  <color rgba="1 0 0 1"/>
+</material>
 </robot>

File: src/rl12dof_urdf_description/urdf/rl12dof_links_joints_hardware.xacro (robot description, xacro)
@@ -2,44 +2,5 @@
 <robot xmlns:xacro="http://www.ros.org/wiki/xacro">
   <xacro:macro name="rl12dof_links_joints" params="">
-    <!-- ========================= -->
-    <!-- TEST STAND LINK           -->
-    <!-- ========================= -->
-    <link name="test_stand">
-      <inertial>
-        <origin xyz="0 0 0.25"/>
-        <mass value="200.0"/>
-        <inertia ixx="5000.0" iyy="5000.0" izz="5000.0" ixy="0" ixz="0" iyz="0"/>
-      </inertial>
-      <visual>
-        <origin xyz="0 0 0.25"/>
-        <geometry>
-          <box size="0.01 0.01 0.5"/>
-        </geometry>
-        <material name="blue"/>
-      </visual>
-      <collision>
-        <origin xyz="0 0 0.25"/>
-        <geometry>
-          <box size="0.01 0.01 0.5"/>
-        </geometry>
-      </collision>
-    </link>
-    <link name="hip_mount">
-      <inertial>
-        <origin xyz="0 0 0"/>
-        <mass value="0.0001"/>
-        <inertia
-          ixx="1e-6" ixy="0" ixz="0"
-          iyy="1e-6" iyz="0"
-          izz="1e-6"/>
-      </inertial>
-      <visual>
-        <geometry>
-          <box size="0.015 0.015 0.015"/>
-        </geometry>
-        <material name="red"/>
-      </visual>
-    </link>
-    <!-- keep everything below here -->
+    <!-- Links -->
     <link name="base_link">
       <inertial>
@@ -283,24 +244,4 @@
     </link>
     <!-- Joints (3 actuated + fixed ones) -->
-    <!-- Have to remove this for hardware -->
-    <!-- <joint name="stand_to_base" type="fixed">
-      <origin xyz="0 0 0.55" rpy="0 -1.5708 0"/>
-      <parent link="test_stand"/>
-      <child link="base_link"/>
-    </joint> -->
-    <!-- To convert stand to a slider -->
-    <joint name="test_stand_slider" type="prismatic">
-      <parent link="test_stand"/>
-      <child link="hip_mount"/>
-      <origin xyz="0 0 0.5" rpy="0 0 0"/>
-      <axis xyz="0 0 -1"/>
-      <limit lower="0" upper="0.50" effort="5000" velocity="0.1"/>
-      <dynamics damping="1.0" friction="0.2"/>
-    </joint>
-    <joint name="base_to_mount" type="fixed">
-      <parent link="hip_mount"/>
-      <child link="base_link"/>
-      <origin xyz="0 0 0" rpy="0 -1.5708 0"/>
-    </joint>
     <joint name="link1_to_base" type="continuous">
       <origin xyz="0.0 0.0 0.007807" rpy="0 0 0"/>

File: src/rl12dof_urdf_description/urdf/rl12dof_urdf.gazebo.xacro (robot description, xacro)
@@ -13,5 +13,5 @@
         <robot_param_node>robot_state_publisher</robot_param_node>
       </plugin>
-      <!-- Optional pose publisher -->
+      <!-- pose publisher -->
       <plugin
         filename="gz-sim-pose-publisher-system"
@@ -19,4 +19,14 @@
         <publish_link_pose>true</publish_link_pose>
       </plugin>
+    </gazebo>
+    <gazebo reference="test_stand">
+      <static>true</static>
+    </gazebo>
+    <gazebo reference="test_stand_slider">
+      <physics>
+        <implicit_spring_damper>true</implicit_spring_damper>
+        <cfm>0</cfm>
+        <erp>1</erp>
+      </physics>
     </gazebo>
     <gazebo reference="link1_to_base">
