Commit message: clean up

File: src/rl12dof_urdf_description/urdf/rl12dof_links_joints.xacro (robot description, xacro)
@@ -301,5 +301,5 @@
       <child link="Foot_V3_Foot_v1_1"/>
     </joint>
-     <gazebo reference="link1_to_base">
+    <!-- <gazebo reference="link1_to_base">
       <joint>
         <type>revolute</type>
@@ -324,5 +324,5 @@
         </axis>
       </joint>
-    </gazebo>
+    </gazebo> -->
   </xacro:macro>
 </robot>

File: src/rl12dof_urdf_description/urdf/rl12dof_urdf.gazebo.xacro (robot description, xacro)
@@ -2,4 +2,5 @@
 <robot xmlns:xacro="http://www.ros.org/wiki/xacro">
   <xacro:macro name="rl12dof_gazebo" params="">
+    <!-- Existing Gazebo plugin block -->
     <gazebo>
       <plugin
@@ -19,4 +20,28 @@
       </plugin>
     </gazebo>
+    <gazebo reference="link1_to_base">
+      <joint>
+        <type>revolute</type>
+        <axis>
+          <xyz>0 0 1</xyz>
+        </axis>
+      </joint>
+    </gazebo>
+    <gazebo reference="link2_to_link1">
+      <joint>
+        <type>revolute</type>
+        <axis>
+          <xyz>0 -1 0</xyz>
+        </axis>
+      </joint>
+    </gazebo>
+    <gazebo reference="link3_to_link2">
+      <joint>
+        <type>revolute</type>
+        <axis>
+          <xyz>0 1 0</xyz>
+        </axis>
+      </joint>
+    </gazebo>
   </xacro:macro>
 </robot>

File: src/rl12dof_urdf_description/urdf/rl12dof_urdf.xacro (robot description, xacro)
@@ -5,5 +5,5 @@
   <!-- Geometry + kinematics -->
   <xacro:include filename="$(find rl12dof_urdf_description)/urdf/rl12dof_links_joints.xacro" />
-  <!-- ros2_control macro (THIS WAS MISSING OR WRONG) -->
+  <!-- ros2_control macro -->
   <xacro:include filename="$(find rl12dof_urdf_description)/urdf/rl12dof_urdf.ros2control.xacro" />
   <!-- Gazebo plugin macro -->
@@ -11,4 +11,10 @@
   <!-- Insert links + joints -->
   <xacro:rl12dof_links_joints />
+  <!-- Fixed joint to world, for SIM ONLY -->
+  <!-- <joint name="base_to_world" type="fixed">
+      <parent link="world"/>
+      <child link="base_link"/>
+      <origin xyz="0 0 0.5" rpy="0 0 0"/>
+  </joint> -->
   <!-- Insert ros2_control block -->
   <xacro:rl12dof_ros2_control />

Commit message: leg move cycle testing

File: src/rl12dof_urdf_description/urdf/rl12dof_links_joints.xacro (robot description, xacro)
@@ -2,4 +2,24 @@
 <robot xmlns:xacro="http://www.ros.org/wiki/xacro">
   <xacro:macro name="rl12dof_links_joints" params="">
+    <link name="test_stand">
+      <inertial>
+        <origin xyz="0 0 0.25" rpy="0 0 0"/>
+        <mass value="200.0"/>
+        <inertia ixx="40.0" iyy="40.0" izz="40.0" ixy="0" ixz="0" iyz="0"/>
+      </inertial>
+      <visual>
+        <origin xyz="0 0 0.25" rpy="0 0 0"/>
+        <geometry>
+          <box size="0.01 0.01 0.5"/> <!-- 1cm x 1cm x 50cm stand -->
+        </geometry>
+        <material name="blue"/>
+      </visual>
+      <collision>
+        <origin xyz="0 0 0.25" rpy="0 0 0"/>
+        <geometry>
+          <box size="0.01 0.01 0.5"/>
+        </geometry>
+      </collision>
+    </link>
     <link name="base_link">
       <inertial>
@@ -243,4 +263,10 @@
     </link>
     <!-- Joints (3 actuated + fixed ones) -->
+    <!-- Have to remove this for hardware -->
+    <joint name="stand_to_base" type="fixed">
+      <origin xyz="0 0 0.55" rpy="0 -1.5708 0"/>
+      <parent link="test_stand"/>
+      <child link="base_link"/>
+    </joint>
     <joint name="link1_to_base" type="continuous">
       <origin xyz="0.0 0.0 0.007807" rpy="0 0 0"/>
@@ -284,5 +310,5 @@
       <parent link="Right_Femur_Housing_v1_1"/>
       <child link="Tibia_Link_v97_1"/>
-      <axis xyz="0.0 1.0 0.0"/>
+      <axis xyz="0.0 -1.0 0.0"/>
     </joint>
     <joint name="drive_to_M3" type="fixed">
@@ -301,28 +327,4 @@
       <child link="Foot_V3_Foot_v1_1"/>
     </joint>
-    <!-- <gazebo reference="link1_to_base">
-      <joint>
-        <type>revolute</type>
-        <axis>
-          <xyz>0 0 1</xyz>
-        </axis>
-      </joint>
-    </gazebo>
-    <gazebo reference="link2_to_link1">
-      <joint>
-        <type>revolute</type>
-        <axis>
-          <xyz>0 -1 0</xyz>
-        </axis>
-      </joint>
-    </gazebo>
-    <gazebo reference="link3_to_link2">
-      <joint>
-        <type>revolute</type>
-        <axis>
-          <xyz>0 1 0</xyz>
-        </axis>
-      </joint>
-    </gazebo> -->
   </xacro:macro>
 </robot>

File: src/rl12dof_urdf_description/urdf/rl12dof_urdf.xacro (robot description, xacro)
@@ -11,10 +11,4 @@
   <!-- Insert links + joints -->
   <xacro:rl12dof_links_joints />
-  <!-- Fixed joint to world, for SIM ONLY -->
-  <!-- <joint name="base_to_world" type="fixed">
-      <parent link="world"/>
-      <child link="base_link"/>
-      <origin xyz="0 0 0.5" rpy="0 0 0"/>
-  </joint> -->
   <!-- Insert ros2_control block -->
   <xacro:rl12dof_ros2_control />

Commit message: increase inertia of stand

File: src/rl12dof_urdf_description/urdf/rl12dof_links_joints.xacro (robot description, xacro)
@@ -6,5 +6,5 @@
         <origin xyz="0 0 0.25" rpy="0 0 0"/>
         <mass value="200.0"/>
-        <inertia ixx="40.0" iyy="40.0" izz="40.0" ixy="0" ixz="0" iyz="0"/>
+        <inertia ixx="100.0" iyy="100.0" izz="100.0" ixy="0" ixz="0" iyz="0"/>
       </inertial>
       <visual>

Commit message: rod is static slider now

File: src/rl12dof_urdf_description/urdf/rl12dof_links_joints.xacro (robot description, xacro)
@@ -12,5 +12,5 @@
       </inertial>
       <visual>
-        <origin xyz="0 0 0.25"/>
+        <origin xyz="0 0 0"/>
         <geometry>
           <box size="0.01 0.01 0.5"/>
@@ -19,9 +19,12 @@
       </visual>
       <collision>
-        <origin xyz="0 0 0.25"/>
+        <origin xyz="0 0 0"/>
         <geometry>
           <box size="0.01 0.01 0.5"/>
         </geometry>
       </collision>
+      <gazebo>
+        <static>true</static>
+      </gazebo>
     </link>
     <link name="hip_mount">
@@ -283,15 +286,9 @@
     </link>
     <!-- Joints (3 actuated + fixed ones) -->
-    <!-- Have to remove this for hardware -->
-    <!-- <joint name="stand_to_base" type="fixed">
-      <origin xyz="0 0 0.55" rpy="0 -1.5708 0"/>
-      <parent link="test_stand"/>
-      <child link="base_link"/>
-    </joint> -->
     <!-- To convert stand to a slider -->
     <joint name="test_stand_slider" type="prismatic">
       <parent link="test_stand"/>
       <child link="hip_mount"/>
-      <origin xyz="0 0 0.5" rpy="0 0 0"/>
+      <origin xyz="0 0 0.25" rpy="0 0 0"/>
       <axis xyz="0 0 -1"/>
       <limit lower="0" upper="0.50" effort="5000" velocity="0.1"/>

File: src/rl12dof_urdf_description/urdf/rl12dof_urdf.gazebo.xacro (robot description, xacro)
@@ -20,6 +20,9 @@
       </plugin>
     </gazebo>
-    <gazebo reference="test_stand">
-      <static>true</static>
+    <gazebo>
+      <joint name="stand_to_world" type="fixed">
+        <parent>world</parent>
+        <child>test_stand</child>
+      </joint>
     </gazebo>
     <gazebo reference="test_stand_slider">
